Commit message: removed the bowl from the world, fixed the camera position by 90 degrees, added the CAD but it is still out of master welding

File: urdf/rs200_simulation.xacro (robot description, xacro)
@@ -10,5 +10,5 @@
     <!-- Create camera instance -->
     <xacro:realsense-rs200 prefix="" parent="world">
-        <origin xyz="0 0 2.0" rpy="0 1.5 0" />
+        <origin xyz="0 0 2.0" rpy="0 1.570796326 0" />
     </xacro:realsense-rs200>
 </robot>
